Commit message: Fixed incorrect and missing dependencies

File: prl_ur5_description/urdf/workbench_ur5.urdf.xacro (robot description, xacro)
@@ -2,5 +2,5 @@
 <robot name="ur5" xmlns:xacro="http://wiki.ros.org/xacro">
   <!-- Load the setup file -->
-  <xacro:property name="setup_file" value="${xacro.load_yaml('$(find prl_ur5_configuration)/config/standart_setup.yaml')}"/>
+  <xacro:property name="setup_file" value="${xacro.load_yaml('$(find prl_ur5_robot_configuration)/config/standart_setup.yaml')}"/>
   <!-- ur5 arm -->
   <xacro:include filename="$(find prl_ur5_description)/urdf/ur5_complete_arm.urdf.xacro"/>
@@ -29,5 +29,5 @@
   <!-- Cameras fixtures (if any) -->
   <xacro:if value="${setup_file.get('fixed_cameras_file') is not None}">
-    <xacro:fixed_cameras parent="prl_ur5_base" fixed_cameras_file="$(find prl_ur5_configuration)/config/${setup_file['fixed_cameras_file']}" turn_on="false"/>
+    <xacro:fixed_cameras parent="prl_ur5_base" fixed_cameras_file="$(find prl_ur5_robot_configuration)/config/${setup_file['fixed_cameras_file']}" turn_on="false"/>
   </xacro:if>
   <!-- back wall -->
@@ -79,6 +79,6 @@
                  gripper_pose="${left.get('gripper_pose')}"
                  hardware_interface="hardware_interface/PositionJointInterface"
-                 joint_limits_parameters_file="$(find prl_ur5_configuration)/config/${left.get('arm_joint_limits')}"
-                 kinematics_parameters_file="$(find prl_ur5_configuration)/config/${left.get('arm_kinematics')}"
+                 joint_limits_parameters_file="$(find prl_ur5_robot_configuration)/config/${left.get('arm_joint_limits')}"
+                 kinematics_parameters_file="$(find prl_ur5_robot_configuration)/config/${left.get('arm_kinematics')}"
                  />
   <!-- Right Arm -->
@@ -91,6 +91,6 @@
                  gripper_pose="${right.get('gripper_pose')}"
                  hardware_interface="hardware_interface/PositionJointInterface"
-                 joint_limits_parameters_file="$(find prl_ur5_configuration)/config/${right.get('arm_joint_limits')}"
-                 kinematics_parameters_file="$(find prl_ur5_configuration)/config/${right.get('arm_kinematics')}"
+                 joint_limits_parameters_file="$(find prl_ur5_robot_configuration)/config/${right.get('arm_joint_limits')}"
+                 kinematics_parameters_file="$(find prl_ur5_robot_configuration)/config/${right.get('arm_kinematics')}"
                  />
   <!-- Linking Arms to world -->
