Commit message: architectural review and doc add

File: prl_ur5_description/urdf/_force_sensor.urdf.xacro (robot description, xacro)
@@ -6,4 +6,5 @@
                         prefix:=''
                         parent:=''
+                        gz_sim:='false'
                         ">
         <!-- force sensor -->
@@ -11,4 +12,41 @@
             <origin xyz="0 0 0" rpy="0 0 ${-pi}"/>
         </xacro:robotiq_ft300>
+        <xacro:if value="${gz_sim}">
+            <!-- enable force_torque sensor -->
+            <gazebo reference="${prefix}measurment_joint">
+                <preserveFixedJoint>true</preserveFixedJoint>
+                <sensor name="${prefix}robotiq_ft_sensor" type="force_torque">
+                    <always_on>true</always_on>
+                    <update_rate>100.0</update_rate>
+                    <visualize>true</visualize>
+                    <topic>${prefix}force_torque</topic>
+                    <force_torque>
+                        <frame>sensor</frame>
+                        <measure_direction>child_to_parent</measure_direction>
+                    </force_torque>
+                </sensor>
+            </gazebo>
+            <gazebo>
+                <plugin filename="ignition-gazebo-forcetorque-system" name="ignition::gazebo::systems::ForceTorque">
+                    <updateRate>100.0</updateRate>
+                    <topicName>${prefix}ft_wrench</topicName>
+                    <jointName>${prefix}measurment_joint</jointName>
+                    <noise>
+                    <type>gaussian</type>
+                    <mean>0.0</mean>
+                    <stddev>0.003</stddev>
+                    </noise>
+                </plugin>
+            </gazebo>
+            <!-- override link properties -->
+            <gazebo reference="${prefix}ft300_sensor">
+                <material>Gazebo/Black</material>
+                <selfCollide>true</selfCollide>
+            </gazebo>
+            <gazebo reference="${prefix}ft300_mounting_plate">
+                <material>Gazebo/Grey</material>
+                <selfCollide>true</selfCollide>
+            </gazebo>
+            </xacro:if>
     </xacro:macro>
 </robot>

File: prl_ur5_description/urdf/_gripper.urdf.xacro (robot description, xacro)
@@ -3,6 +3,4 @@
   <!-- onrobot RG2(6) -->
   <xacro:include filename="$(find onrobot_description)/urdf/onrobot_rg.urdf.xacro"/>
-  <!-- weiss wsg50-->
-  <xacro:include filename="$(find wsg50_simulation)/urdf/wsg_50.urdf.xacro"/>
   <xacro:macro name="gripper" params="gripper prefix parent pose hardware_interface gz_sim">
     <!-- check gripper type -->
@@ -30,4 +28,5 @@
     <!-- if weiss-wsg50 -->
     <xacro:if value="${gripper == 'weiss-wsg50'}">
+      <xacro:include filename="$(find wsg50_simulation)/urdf/wsg_50.urdf.xacro"/>
       <xacro:wsg_50_xacro name="${prefix}wsg50" parent="${parent}" finger_length="0.023" finger_tip="0.0">
         <origin xyz="${pose['x']} ${pose['y']} ${pose['z']}" rpy="${pose['roll']} ${pose['pitch']} ${pose['yaw']}"/>

File: prl_ur5_description/urdf/ur5_complete_arm.urdf.xacro (robot description, xacro)
@@ -1,68 +1,92 @@
 <?xml version="1.0"?>
 <robot xmlns:xacro="http://wiki.ros.org/xacro">
-  <!-- ur5 -->
-  <xacro:include filename="$(find prl_ur5_description)/urdf/ur5_macro.xacro" />
-  <!-- Force sensor -->
-  <xacro:include filename="$(find prl_ur5_description)/urdf/_force_sensor.urdf.xacro" />
-  <!-- gripper -->
-  <xacro:include filename="$(find prl_ur5_description)/urdf/_gripper.urdf.xacro"/>
-  <xacro:macro name="ur5" params="
-      prefix
-      parent
-      pose
-      sensor
-      hardware_interface
-      gz_sim:=False
-      gripper:=None
-      gripper_pose:=None
-      camera:=None
-      camera_pose:=None
-      joint_limits_parameters_file:='$(find ur_description)/config/ur5/joint_limits.yaml'
-      kinematics_parameters_file:='$(find ur_description)/config/ur5/default_kinematics.yaml'
-      transmission_hw_interface:=hardware_interface/PositionJointInterface
-    ">
     <!-- ur5 -->
-    <xacro:ur5_robot
-      prefix="${prefix}"
-      parent="${parent}"
-      pose="${pose}"
-      transmission_hw_interface="${hardware_interface}"
-      gz_sim="${gz_sim}"
-      joint_limits_parameters_file="${joint_limits_parameters_file}"
-      kinematics_parameters_file="${kinematics_parameters_file}"
-      />
-    <!-- force sensor -->
-    <xacro:force_sensor
-        prefix='${prefix}'
-        parent="tool0"
-    />
-    <!-- tool frame -->
-    <link name="${prefix}tool"/>
-    <joint name="${prefix}tool_joint" type="fixed">
-      <origin xyz="0 0 0" rpy="0 0 ${-pi}"/>
-      <parent link="${prefix}robotiq_ft_frame_id"/>
-      <child link="${prefix}tool"/>
-    </joint>
+    <xacro:include filename="$(find ur_description)/urdf/ur_macro.xacro"/>
+    <xacro:include filename="$(find ur_description)/urdf/inc/ur_joint_control.xacro" />
+    <!-- force sensor-->
+    <xacro:include filename="$(find prl_ur5_description)/urdf/_force_sensor.urdf.xacro"/>
     <!-- gripper -->
-    <xacro:gripper gripper="${gripper}" prefix='${prefix}' parent="${prefix}tool" pose="${gripper_pose}" hardware_interface="${hardware_interface}" gz_sim="${gz_sim}"/>
-    <!-- Right angle connector -->
-    <link name="${prefix}wrist_connector_link">
-      <visual>
-          <geometry>
-              <mesh filename="package://prl_ur5_description/model/RG_connector_simple.stl"/>
-          </geometry>
-          <material name="connector_green"><color rgba="0.2 0.8 0 1"/></material>
-      </visual>
-      <collision>
-          <geometry>
-              <mesh filename="package://prl_ur5_description/model/RG_connector_simple_convex.stl"/>
-          </geometry>
-      </collision>
-    </link>
-    <joint name="${prefix}wrist_connector" type="fixed">
-      <origin xyz="0 -0.0375 -0.02" rpy="1.5708 0 0"/>
-      <parent link="${prefix}wrist_3_link"/>
-      <child link="${prefix}wrist_connector_link"/>
-    </joint>
-  </xacro:macro>
+    <xacro:include filename="$(find prl_ur5_description)/urdf/_gripper.urdf.xacro"/>
+    <xacro:macro name="ur5" params="
+        name:=ur
+        ur_type:=ur5
+        prefix
+        parent
+        pose
+        sensor
+        gripper
+        gripper_pose
+        joint_limits_parameters_file:='$(find ur_description)/config/ur5/joint_limits.yaml'
+        kinematics_parameters_file:='$(find ur_description)/config/ur5/default_kinematics.yaml'
+        hw_interface:=hardware_interface/PositionJointInterface
+        physical_parameters_file:='$(find ur_description)/config/ur5/physical_parameters.yaml'
+        visual_parameters_file:='$(find ur_description)/config/ur5/visual_parameters.yaml'
+        safety_limits:=false
+        safety_pos_margin:=0.15
+        safety_k_position:=20
+        gz_sim:=false
+        ros2_control:=false
+        ">
+        <xacro:ur_robot
+            name="${prefix}ur"
+            tf_prefix="${prefix}"
+            parent="${parent}"
+            joint_limits_parameters_file="${joint_limits_parameters_file}"
+            kinematics_parameters_file="${kinematics_parameters_file}"
+            physical_parameters_file="${physical_parameters_file}"
+            visual_parameters_file="${visual_parameters_file}"
+            safety_limits="${safety_limits}"
+            safety_pos_margin="${safety_pos_margin}"
+            safety_k_position="${safety_k_position}"
+            force_abs_paths="${gz_sim}"
+        >
+        <origin xyz="${pose['x']} ${pose['y']} ${pose['z']}" rpy="${pose['roll']} ${pose['pitch']} ${pose['yaw']}"/>
+        </xacro:ur_robot>
+        <xacro:if value="${gz_sim or ros2_control}">
+             <!-- ros2 control instance -->
+            <ros2_control name="${prefix}ur" type="system">
+                <hardware>
+                    <plugin>gz_ros2_control/GazeboSimSystem</plugin>
+                </hardware>
+                <xacro:ur_joint_control_description
+                    tf_prefix="${prefix}"
+                    initial_positions="${dict(shoulder_pan_joint=0.0,shoulder_lift_joint=-1.57,elbow_joint=0.0,wrist_1_joint=-1.57,wrist_2_joint=0.0,wrist_3_joint=0.0)}"
+                />
+            </ros2_control>
+        </xacro:if>
+        <!-- force sensor -->
+        <xacro:force_sensor
+            prefix="${prefix}"
+            parent="tool0"
+            gz_sim="${gz_sim}"
+        />
+        <!-- tool frame -->
+        <link name="${prefix}tool"/>
+        <joint name="${prefix}tool_joint" type="fixed">
+            <origin xyz="0 0 0" rpy="0 0 ${-pi}"/>
+            <parent link="${prefix}robotiq_ft_frame_id"/>
+            <child link="${prefix}tool"/>
+        </joint>
+        <!-- gripper -->
+        <xacro:gripper gripper="${gripper}" prefix='${prefix}' parent="${prefix}tool" pose="${gripper_pose}" hardware_interface="${hw_interface}" gz_sim="${gz_sim}"/>
+        <!-- Right angle connector -->
+        <link name="${prefix}wrist_connector_link">
+        <visual>
+            <geometry>
+                <mesh filename="file://$(find prl_ur5_description)/model/RG_connector_simple.stl"/>
+            </geometry>
+            <material name="connector_green"><color rgba="0.2 0.8 0 1"/></material>
+        </visual>
+        <collision>
+            <geometry>
+                <mesh filename="file://$(find prl_ur5_description)/model/RG_connector_simple_convex.stl"/>
+            </geometry>
+        </collision>
+        </link>
+        <joint name="${prefix}wrist_connector" type="fixed">
+        <origin xyz="0 -0.0375 -0.02" rpy="1.5708 0 0"/>
+        <parent link="${prefix}wrist_3_link"/>
+        <child link="${prefix}wrist_connector_link"/>
+        </joint>
+    </xacro:macro>
 </robot>

File: prl_ur5_description/urdf/workbench_ur5.urdf.xacro (robot description, xacro)
@@ -1,4 +1,6 @@
 <?xml version="1.0"?>
-<robot name="ur5" xmlns:xacro="http://wiki.ros.org/xacro">
+<robot xmlns:xacro="http://wiki.ros.org/xacro" name="ur5" >
+  <xacro:arg name="controller_file" default="$(find prl_ur5_control)/config/dual_ur_controller.yaml"/>
+  <xacro:arg name="gz_sim" default="false"/>
   <!-- Load the setup file -->
   <xacro:property name="setup_file" value="${xacro.load_yaml('$(find prl_ur5_robot_configuration)/config/standart_setup.yaml')}"/>
@@ -7,6 +9,9 @@
   <!-- fixed camera-->
   <xacro:include filename="$(find prl_ur5_description)/urdf/_fixed_cameras.urdf.xacro"/>
-  <!-- Global frame -->
+  <!-- Repere global -->
   <link name="prl_ur5_base"/>
+  <gazebo >
+    <selfCollide>true</selfCollide>
+  </gazebo>
   <!-- Table -->
   <link name="table_link">
@@ -15,4 +20,5 @@
         <mesh filename="file://$(find prl_ur5_description)/model/vention_table.stl"/>
       </geometry>
+      <material name="red"><color rgba="1 0 0 1"/></material>
     </visual>
     <collision>
@@ -29,5 +35,5 @@
   <!-- Cameras fixtures (if any) -->
   <xacro:if value="${setup_file.get('fixed_cameras_file') is not None}">
-    <xacro:fixed_cameras parent="prl_ur5_base" fixed_cameras_file="$(find prl_ur5_robot_configuration)/config/${setup_file['fixed_cameras_file']}" turn_on="false"/>
+    <xacro:fixed_cameras parent="prl_ur5_base" fixed_cameras_file="$(find prl_ur5_robot_configuration)/config/${setup_file['fixed_cameras_file']}" turn_on="true"/>
   </xacro:if>
   <!-- back wall -->
@@ -76,7 +82,7 @@
                  pose="${left['arm_pose']}"
                  sensor="false"
-                 gripper="weiss-wsg50"
+                 gz_sim="$(arg gz_sim)"
+                 gripper="${left.get('gripper')}"
                  gripper_pose="${left.get('gripper_pose')}"
-                 hardware_interface="hardware_interface/PositionJointInterface"
                  joint_limits_parameters_file="$(find prl_ur5_robot_configuration)/config/${left.get('arm_joint_limits')}"
                  kinematics_parameters_file="$(find prl_ur5_robot_configuration)/config/${left.get('arm_kinematics')}"
@@ -88,10 +94,17 @@
                  pose="${right['arm_pose']}"
                  sensor="false"
-                 gripper="weiss-wsg50"
+                 gz_sim="$(arg gz_sim)"
+                 gripper="${right.get('gripper')}"
                  gripper_pose="${right.get('gripper_pose')}"
-                 hardware_interface="hardware_interface/PositionJointInterface"
                  joint_limits_parameters_file="$(find prl_ur5_robot_configuration)/config/${right.get('arm_joint_limits')}"
                  kinematics_parameters_file="$(find prl_ur5_robot_configuration)/config/${right.get('arm_kinematics')}"
                  />
+  <xacro:if value="$(arg gz_sim)">
+    <gazebo>
+        <plugin filename="gz_ros2_control-system" name="gz_ros2_control::GazeboSimROS2ControlPlugin">
+        <parameters>$(arg controller_file)</parameters>
+        </plugin>
+    </gazebo>
+  </xacro:if>
   <!-- Linking Arms to world -->
   <link name="base_link" />

Commit message: review fix

File: prl_ur5_description/urdf/_force_sensor.urdf.xacro (robot description, xacro)
@@ -28,5 +28,5 @@
             </gazebo>
             <gazebo>
-                <plugin filename="ignition-gazebo-forcetorque-system" name="ignition::gazebo::systems::ForceTorque">
+                <plugin filename="gz-sim-forcetorque-system" name="gz::sim::systems::ForceTorque">
                     <updateRate>100.0</updateRate>
                     <topicName>${prefix}ft_wrench</topicName>

File: prl_ur5_description/urdf/_gripper.urdf.xacro (robot description, xacro)
@@ -27,10 +27,10 @@
     </xacro:if>
     <!-- if weiss-wsg50 -->
-    <xacro:if value="${gripper == 'weiss-wsg50'}">
+    <!-- <xacro:if value="${gripper == 'weiss-wsg50'}">
       <xacro:include filename="$(find wsg50_simulation)/urdf/wsg_50.urdf.xacro"/>
       <xacro:wsg_50_xacro name="${prefix}wsg50" parent="${parent}" finger_length="0.023" finger_tip="0.0">
         <origin xyz="${pose['x']} ${pose['y']} ${pose['z']}" rpy="${pose['roll']} ${pose['pitch']} ${pose['yaw']}"/>
       </xacro:wsg_50_xacro>
-    </xacro:if>
+    </xacro:if> -->
     <!-- if allegro-hand -->
     <!-- <xacro:if value="${gripper.startswith('allegro-hand:')}">

File: prl_ur5_description/urdf/ur5_complete_arm.urdf.xacro (robot description, xacro)
@@ -61,32 +61,4 @@
             gz_sim="${gz_sim}"
         />
-        <!-- tool frame -->
-        <link name="${prefix}tool"/>
-        <joint name="${prefix}tool_joint" type="fixed">
-            <origin xyz="0 0 0" rpy="0 0 ${-pi}"/>
-            <parent link="${prefix}robotiq_ft_frame_id"/>
-            <child link="${prefix}tool"/>
-        </joint>
-        <!-- gripper -->
-        <xacro:gripper gripper="${gripper}" prefix='${prefix}' parent="${prefix}tool" pose="${gripper_pose}" hardware_interface="${hw_interface}" gz_sim="${gz_sim}"/>
-        <!-- Right angle connector -->
-        <link name="${prefix}wrist_connector_link">
-        <visual>
-            <geometry>
-                <mesh filename="file://$(find prl_ur5_description)/model/RG_connector_simple.stl"/>
-            </geometry>
-            <material name="connector_green"><color rgba="0.2 0.8 0 1"/></material>
-        </visual>
-        <collision>
-            <geometry>
-                <mesh filename="file://$(find prl_ur5_description)/model/RG_connector_simple_convex.stl"/>
-            </geometry>
-        </collision>
-        </link>
-        <joint name="${prefix}wrist_connector" type="fixed">
-        <origin xyz="0 -0.0375 -0.02" rpy="1.5708 0 0"/>
-        <parent link="${prefix}wrist_3_link"/>
-        <child link="${prefix}wrist_connector_link"/>
-        </joint>
     </xacro:macro>
 </robot>

File: prl_ur5_description/urdf/workbench_ur5.urdf.xacro (robot description, xacro)
@@ -11,8 +11,8 @@
   <!-- Repere global -->
   <link name="prl_ur5_base"/>
-  <gazebo >
-    <selfCollide>true</selfCollide>
-  </gazebo>
   <!-- Table -->
+  <material name="Blue">
+    <color rgba="${0/255} ${30/255} ${70/255} 1.0"/>
+  </material>
   <link name="table_link">
     <visual>
@@ -20,5 +20,5 @@
         <mesh filename="file://$(find prl_ur5_description)/model/vention_table.stl"/>
       </geometry>
-      <material name="red"><color rgba="1 0 0 1"/></material>
+      <material name="Blue"/>
     </visual>
     <collision>
