Commit message: modification after the PR review

File: prl_ur5_description/urdf/ur5_complete_arm.urdf.xacro (robot description, xacro)
@@ -4,9 +4,7 @@
   <xacro:include filename="$(find prl_ur5_description)/urdf/ur5_macro.xacro" />
   <!-- Force sensor -->
-  <xacro:include filename="$(find prl_ur5_description)/urdf/_force_sensor.urdf.xacro"/>
+  <xacro:include filename="$(find robotiq_ft_sensor_description)/urdf/robotiq_ft300.urdf.xacro" />
   <!-- gripper -->
   <xacro:include filename="$(find prl_ur5_description)/urdf/_gripper.urdf.xacro"/>
-  <!-- camera -->
-  <!-- <xacro:include filename="$(find prl_ur5_description)/urdf/_camera_sensor.urdf.xacro"/> -->
   <xacro:macro name="ur5" params="
       prefix
@@ -20,4 +18,7 @@
       camera:=None
       camera_pose:=None
+      joint_limits_parameters_file:='$(find ur_description)/config/ur5/joint_limits.yaml'
+      kinematics_parameters_file:='$(find ur_description)/config/ur5/default_kinematics.yaml'
+      transmission_hw_interface:=hardware_interface/PositionJointInterface
     ">
     <!-- ur5 -->
@@ -28,7 +29,11 @@
       transmission_hw_interface="${hardware_interface}"
       gz_sim="${gz_sim}"
+      joint_limits_parameters_file="${joint_limits_parameters_file}"
+      kinematics_parameters_file="${kinematics_parameters_file}"
       />
     <!-- force sensor -->
-    <xacro:force_sensor prefix='${prefix}' parent="tool0"/>
+    <xacro:robotiq_ft300 tf_prefix="${prefix}" parent="tool0">
+      <origin rpy="0 0 ${-pi/2}" xyz="0 0 -0.004"/>
+    </xacro:robotiq_ft300>
     <!-- tool frame -->
     <link name="${prefix}tool"/>

File: prl_ur5_description/urdf/workbench_ur5.urdf.xacro (robot description, xacro)
@@ -2,9 +2,7 @@
 <robot name="ur5" xmlns:xacro="http://wiki.ros.org/xacro">
   <!-- Load the setup file -->
-  <xacro:property name="setup_file" value="${xacro.load_yaml('$(find prl_ur5_robot_configuration)/config/standart_setup.yaml')}"/>
+  <xacro:property name="setup_file" value="${xacro.load_yaml('$(find prl_ur5_configuration)/config/standart_setup.yaml')}"/>
   <!-- ur5 arm -->
   <xacro:include filename="$(find prl_ur5_description)/urdf/ur5_complete_arm.urdf.xacro"/>
-  <!-- Fixed cameras -->
-  <!-- <xacro:include filename="$(find prl_ur5_description)/urdf/_fixed_cameras.urdf.xacro"/> -->
   <!-- Global frame -->
   <link name="prl_ur5_base"/>
@@ -75,4 +73,6 @@
                  gripper_pose="${left.get('gripper_pose')}"
                  hardware_interface="hardware_interface/PositionJointInterface"
+                 joint_limits_parameters_file="$(find prl_ur5_configuration)/config/${left.get('arm_joint_limits')}"
+                 kinematics_parameters_file="$(find prl_ur5_configuration)/config/${left.get('arm_kinematics')}"
                  />
   <!-- Right Arm -->
@@ -85,4 +85,6 @@
                  gripper_pose="${right.get('gripper_pose')}"
                  hardware_interface="hardware_interface/PositionJointInterface"
+                 joint_limits_parameters_file="$(find prl_ur5_configuration)/config/${left.get('arm_joint_limits')}"
+                 kinematics_parameters_file="$(find prl_ur5_configuration)/config/${left.get('arm_kinematics')}"
                  />
   <!-- Linking Arms to world -->

Commit message: add a clean file to load ft300 sensor

File: prl_ur5_description/urdf/ur5_complete_arm.urdf.xacro (robot description, xacro)
@@ -4,5 +4,5 @@
   <xacro:include filename="$(find prl_ur5_description)/urdf/ur5_macro.xacro" />
   <!-- Force sensor -->
-  <xacro:include filename="$(find robotiq_ft_sensor_description)/urdf/robotiq_ft300.urdf.xacro" />
+  <xacro:include filename="$(find prl_ur5_description)/urdf/_force_sensor.urdf.xacro" />
   <!-- gripper -->
   <xacro:include filename="$(find prl_ur5_description)/urdf/_gripper.urdf.xacro"/>
@@ -33,7 +33,8 @@
       />
     <!-- force sensor -->
-    <xacro:robotiq_ft300 tf_prefix="${prefix}" parent="tool0">
-      <origin rpy="0 0 ${-pi/2}" xyz="0 0 -0.004"/>
-    </xacro:robotiq_ft300>
+    <xacro:force_sensor
+        prefix='${prefix}'
+        parent="tool0"
+    />
     <!-- tool frame -->
     <link name="${prefix}tool"/>
@@ -64,8 +65,4 @@
       <child link="${prefix}wrist_connector_link"/>
     </joint>
-    <!-- hand-eye camera
-    <xacro:unless value="${camera is None}">
-      <xacro:camera_sensor camera="${camera}" prefix='${prefix}' parent="${prefix}tool" pose="${camera_pose}" turn_on="${sensor}"/>
-    </xacro:unless> -->
   </xacro:macro>
 </robot>

File: prl_ur5_description/urdf/workbench_ur5.urdf.xacro (robot description, xacro)
@@ -5,4 +5,6 @@
   <!-- ur5 arm -->
   <xacro:include filename="$(find prl_ur5_description)/urdf/ur5_complete_arm.urdf.xacro"/>
+  <!-- fixed camera-->
+  <xacro:include filename="$(find prl_ur5_description)/urdf/_fixed_cameras.urdf.xacro"/>
   <!-- Global frame -->
   <link name="prl_ur5_base"/>
@@ -25,4 +27,8 @@
     <origin xyz="0.0 0.0 0.0" rpy="0.0 0.0 0.0"/>
   </joint>
+  <!-- Cameras fixtures (if any) -->
+  <xacro:if value="${setup_file.get('fixed_cameras_file') is not None}">
+    <xacro:fixed_cameras parent="prl_ur5_base" fixed_cameras_file="$(find prl_ur5_configuration)/config/${setup_file['fixed_cameras_file']}" turn_on="false"/>
+  </xacro:if>
   <!-- back wall -->
   <link name="backwall_link">

Commit message: Controller update and standardisation of launch file for simulated and real robot

File: prl_ur5_description/urdf/ur5_complete_arm.urdf.xacro (robot description, xacro)
@@ -4,4 +4,5 @@
     <xacro:include filename="$(find ur_description)/urdf/ur_macro.xacro"/>
     <xacro:include filename="$(find ur_description)/urdf/inc/ur_joint_control.xacro" />
+    <xacro:include filename="$(find ur_robot_driver)/urdf/ur.ros2_control.xacro"/>
     <!-- force sensor-->
     <xacro:include filename="$(find prl_ur5_description)/urdf/_force_sensor.urdf.xacro"/>
@@ -26,5 +27,10 @@
         safety_k_position:=20
         gz_sim:=false
-        ros2_control:=false
+        real_robot:=false
+        headless_mode:=true
+        ur_output_recipe_filename:='$(find ur_robot_driver)/resources/rtde_output_recipe.txt'
+        ur_input_recipe_filename:='$(find ur_robot_driver)/resources/rtde_input_recipe.txt'
+        ur_script_filename:='$(find ur_client_library)/resources/external_control.urscript'
+        network := ''
         ">
         <xacro:ur_robot
@@ -43,6 +49,5 @@
         <origin xyz="${pose['x']} ${pose['y']} ${pose['z']}" rpy="${pose['roll']} ${pose['pitch']} ${pose['yaw']}"/>
         </xacro:ur_robot>
-        <xacro:if value="${gz_sim or ros2_control}">
-             <!-- ros2 control instance -->
+        <xacro:if value="${gz_sim}">
             <ros2_control name="${prefix}ur" type="system">
                 <hardware>
@@ -54,4 +59,22 @@
                 />
             </ros2_control>
+        </xacro:if>
+        <xacro:if value="${real_robot}">
+            <xacro:ur_ros2_control
+                name="${prefix}ur"
+                tf_prefix="${prefix}"
+                kinematics_parameters_file="${kinematics_parameters_file}"
+                robot_ip="${network['ip']}"
+                script_filename="${ur_script_filename}"
+                output_recipe_filename="${ur_output_recipe_filename}"
+                input_recipe_filename="${ur_input_recipe_filename}"
+                use_mock_hardware="false"
+                mock_sensor_commands="false"
+                headless_mode="${headless_mode}"
+                script_command_port="${network['script_command_port']}"
+                reverse_port="${network['reverse_port']}"
+                script_sender_port="${network['script_sender_port']}"
+                trajectory_port="${network['trajectory_port']}"
+            />
         </xacro:if>
         <!-- force sensor -->

File: prl_ur5_description/urdf/workbench_ur5.urdf.xacro (robot description, xacro)
@@ -1,12 +1,14 @@
 <?xml version="1.0"?>
 <robot xmlns:xacro="http://wiki.ros.org/xacro" name="ur5" >
+  <!-- Arguments-->
+  <xacro:arg name="gz_sim" default="false"/>
+  <xacro:arg name="real_robot" default="false"/>
+  <!-- Setup files -->
   <xacro:arg name="controller_file" default="$(find prl_ur5_control)/config/dual_ur_controller.yaml"/>
-  <xacro:arg name="gz_sim" default="false"/>
-  <!-- Load the setup file -->
   <xacro:property name="setup_file" value="${xacro.load_yaml('$(find prl_ur5_robot_configuration)/config/standart_setup.yaml')}"/>
   <!-- ur5 arm -->
   <xacro:include filename="$(find prl_ur5_description)/urdf/ur5_complete_arm.urdf.xacro"/>
   <!-- fixed camera-->
-  <xacro:include filename="$(find prl_ur5_description)/urdf/_fixed_cameras.urdf.xacro"/>
+  <!-- <xacro:include filename="$(find prl_ur5_description)/urdf/_fixed_cameras.urdf.xacro"/> -->
   <!-- Repere global -->
   <link name="prl_ur5_base"/>
@@ -34,7 +36,7 @@
   </joint>
   <!-- Cameras fixtures (if any) -->
-  <xacro:if value="${setup_file.get('fixed_cameras_file') is not None}">
+  <!-- <xacro:if value="${setup_file.get('fixed_cameras_file') is not None}">
     <xacro:fixed_cameras parent="prl_ur5_base" fixed_cameras_file="$(find prl_ur5_robot_configuration)/config/${setup_file['fixed_cameras_file']}" turn_on="true"/>
-  </xacro:if>
+  </xacro:if> -->
   <!-- back wall -->
   <link name="backwall_link">
@@ -87,4 +89,6 @@
                  joint_limits_parameters_file="$(find prl_ur5_robot_configuration)/config/${left.get('arm_joint_limits')}"
                  kinematics_parameters_file="$(find prl_ur5_robot_configuration)/config/${left.get('arm_kinematics')}"
+                 real_robot="$(arg real_robot)"
+                 network = "${left.get('network')}"
                  />
   <!-- Right Arm -->
@@ -99,4 +103,6 @@
                  joint_limits_parameters_file="$(find prl_ur5_robot_configuration)/config/${right.get('arm_joint_limits')}"
                  kinematics_parameters_file="$(find prl_ur5_robot_configuration)/config/${right.get('arm_kinematics')}"
+                 real_robot="$(arg real_robot)"
+                 network = "${right.get('network')}"
                  />
   <xacro:if value="$(arg gz_sim)">

File: prl_ur5_moveit/config/ur5.ros2_control.xacro (robot description, xacro)
@@ -92,29 +92,29 @@
                 <state_interface name="velocity"/>
             </joint>
-            <joint name="left_wsg50_base_joint_gripper_left">
+            <joint name="left_gripper_base_joint_gripper_left">
                 <command_interface name="position"/>
                 <state_interface name="position">
-                  <param name="initial_value">${initial_positions['left_wsg50_base_joint_gripper_left']}</param>
+                  <param name="initial_value">${initial_positions['left_gripper_base_joint_gripper_left']}</param>
                 </state_interface>
                 <state_interface name="velocity"/>
             </joint>
-            <joint name="left_wsg50_base_joint_gripper_right">
+            <joint name="left_gripper_base_joint_gripper_right">
                 <command_interface name="position"/>
                 <state_interface name="position">
-                  <param name="initial_value">${initial_positions['left_wsg50_base_joint_gripper_right']}</param>
+                  <param name="initial_value">${initial_positions['left_gripper_base_joint_gripper_right']}</param>
                 </state_interface>
                 <state_interface name="velocity"/>
             </joint>
-            <joint name="right_wsg50_base_joint_gripper_left">
+            <joint name="right_gripper_base_joint_gripper_left">
                 <command_interface name="position"/>
                 <state_interface name="position">
-                  <param name="initial_value">${initial_positions['right_wsg50_base_joint_gripper_left']}</param>
+                  <param name="initial_value">${initial_positions['right_gripper_base_joint_gripper_left']}</param>
                 </state_interface>
                 <state_interface name="velocity"/>
             </joint>
-            <joint name="right_wsg50_base_joint_gripper_right">
+            <joint name="right_gripper_base_joint_gripper_right">
                 <command_interface name="position"/>
                 <state_interface name="position">
-                  <param name="initial_value">${initial_positions['right_wsg50_base_joint_gripper_right']}</param>
+                  <param name="initial_value">${initial_positions['right_gripper_base_joint_gripper_right']}</param>
                 </state_interface>
                 <state_interface name="velocity"/>

Commit message: pr review
change param and name of ur5 macro
add doc
enable camera visual

File: prl_ur5_description/urdf/ur5_complete_arm.urdf.xacro (robot description, xacro)
@@ -9,5 +9,5 @@
     <!-- gripper -->
     <xacro:include filename="$(find prl_ur5_description)/urdf/_gripper.urdf.xacro"/>
-    <xacro:macro name="ur5" params="
+    <xacro:macro name="arm" params="
         name:=ur
         ur_type:=ur5
@@ -27,5 +27,4 @@
         safety_k_position:=20
         gz_sim:=false
-        real_robot:=false
         headless_mode:=true
         ur_output_recipe_filename:='$(find ur_robot_driver)/resources/rtde_output_recipe.txt'
@@ -60,5 +59,5 @@
             </ros2_control>
         </xacro:if>
-        <xacro:if value="${real_robot}">
+        <xacro:unless value="${gz_sim}">
             <xacro:ur_ros2_control
                 name="${prefix}ur"
@@ -77,5 +76,5 @@
                 trajectory_port="${network['trajectory_port']}"
             />
-        </xacro:if>
+        </xacro:unless>
         <!-- force sensor -->
         <xacro:force_sensor

File: prl_ur5_description/urdf/workbench_ur5.urdf.xacro (robot description, xacro)
@@ -10,5 +10,5 @@
   <xacro:include filename="$(find prl_ur5_description)/urdf/ur5_complete_arm.urdf.xacro"/>
   <!-- fixed camera-->
-  <!-- <xacro:include filename="$(find prl_ur5_description)/urdf/_fixed_cameras.urdf.xacro"/> -->
+  <xacro:include filename="$(find prl_ur5_description)/urdf/_fixed_cameras.urdf.xacro"/>
   <!-- Repere global -->
   <link name="prl_ur5_base"/>
@@ -36,7 +36,7 @@
   </joint>
   <!-- Cameras fixtures (if any) -->
-  <!-- <xacro:if value="${setup_file.get('fixed_cameras_file') is not None}">
+  <xacro:if value="${setup_file.get('fixed_cameras_file') is not None}">
     <xacro:fixed_cameras parent="prl_ur5_base" fixed_cameras_file="$(find prl_ur5_robot_configuration)/config/${setup_file['fixed_cameras_file']}" turn_on="true"/>
-  </xacro:if> -->
+  </xacro:if>
   <!-- back wall -->
   <link name="backwall_link">
@@ -80,5 +80,5 @@
   <!-- Left arm -->
   <xacro:property name="left" value="${setup_file.get('left')}"/>
-  <xacro:ur5 prefix="left_"
+  <xacro:arm prefix="left_"
                  parent="prl_ur5_base"
                  pose="${left['arm_pose']}"
@@ -89,10 +89,9 @@
                  joint_limits_parameters_file="$(find prl_ur5_robot_configuration)/config/${left.get('arm_joint_limits')}"
                  kinematics_parameters_file="$(find prl_ur5_robot_configuration)/config/${left.get('arm_kinematics')}"
-                 real_robot="$(arg real_robot)"
                  network = "${left.get('network')}"
                  />
   <!-- Right Arm -->
   <xacro:property name="right" value="${setup_file.get('right')}"/>
-  <xacro:ur5 prefix="right_"
+  <xacro:arm prefix="right_"
                  parent="prl_ur5_base"
                  pose="${right['arm_pose']}"
@@ -103,5 +102,4 @@
                  joint_limits_parameters_file="$(find prl_ur5_robot_configuration)/config/${right.get('arm_joint_limits')}"
                  kinematics_parameters_file="$(find prl_ur5_robot_configuration)/config/${right.get('arm_kinematics')}"
-                 real_robot="$(arg real_robot)"
                  network = "${right.get('network')}"
                  />

Commit message: add some doc

File: prl_ur5_description/urdf/ur5_complete_arm.urdf.xacro (robot description, xacro)
@@ -10,5 +10,5 @@
     <xacro:include filename="$(find prl_ur5_description)/urdf/_gripper.urdf.xacro"/>
     <!-- Macro to define the complete arm -->
-    <xacro:macro name="ur5" params="
+    <xacro:macro name="arm" params="
         name:=ur
         ur_type:=ur5
@@ -28,5 +28,4 @@
         safety_k_position:=20
         gz_sim:=false
-        real_robot:=false
         headless_mode:=true
         ur_output_recipe_filename:='$(find ur_robot_driver)/resources/rtde_output_recipe.txt'
@@ -64,5 +63,5 @@
         </xacro:if>
         <!-- ROS2 control if real robot -->
-        <xacro:if value="${real_robot}">
+        <xacro:unless value="${gz_sim}">
             <xacro:ur_ros2_control
                 name="${prefix}ur"
@@ -81,5 +80,5 @@
                 trajectory_port="${network['trajectory_port']}"
             />
-        </xacro:if>
+        </xacro:unless>
         <!-- Force sensor -->
         <xacro:force_sensor

File: prl_ur5_description/urdf/workbench_ur5.urdf.xacro (robot description, xacro)
@@ -1,4 +1,4 @@
 <?xml version="1.0"?>
-<robot xmlns:xacro="http://wiki.ros.org/xacro" name="ur5" >
+<robot xmlns:xacro="http://wiki.ros.org/xacro" name="bimanual_robot" >
   <!-- Arguments-->
   <xacro:arg name="gz_sim" default="false"/>
@@ -80,5 +80,5 @@
   <!-- Left arm -->
   <xacro:property name="left" value="${setup_file.get('left')}"/>
-  <xacro:ur5 prefix="left_"
+  <xacro:arm prefix="left_"
                  parent="prl_ur5_base"
                  pose="${left['arm_pose']}"
@@ -89,10 +89,9 @@
                  joint_limits_parameters_file="$(find prl_ur5_robot_configuration)/config/${left.get('arm_joint_limits')}"
                  kinematics_parameters_file="$(find prl_ur5_robot_configuration)/config/${left.get('arm_kinematics')}"
-                 real_robot="$(arg real_robot)"
                  network = "${left.get('network')}"
                  />
   <!-- Right Arm -->
   <xacro:property name="right" value="${setup_file.get('right')}"/>
-  <xacro:ur5 prefix="right_"
+  <xacro:arm prefix="right_"
                  parent="prl_ur5_base"
                  pose="${right['arm_pose']}"
@@ -103,5 +102,4 @@
                  joint_limits_parameters_file="$(find prl_ur5_robot_configuration)/config/${right.get('arm_joint_limits')}"
                  kinematics_parameters_file="$(find prl_ur5_robot_configuration)/config/${right.get('arm_kinematics')}"
-                 real_robot="$(arg real_robot)"
                  network = "${right.get('network')}"
                  />
