Commit message: adding wsg50 gripper

File: prl_ur5_description/urdf/_gripper.urdf.xacro (robot description, xacro)
@@ -3,7 +3,9 @@
   <!-- onrobot RG2(6) -->
   <xacro:include filename="$(find onrobot_description)/urdf/onrobot_rg.urdf.xacro"/>
+  <!-- weiss wsg50-->
+  <xacro:include filename="$(find wsg_50_simulation)/urdf/wsg_50.urdf.xacro"/>
   <xacro:macro name="gripper" params="gripper prefix parent pose hardware_interface gz_sim">
     <!-- check gripper type -->
-    <xacro:unless value="${gripper in [None, 'onrobot-rg2', 'onrobot-rg6', 'onrobot-rg6-v2'] or gripper.startswith('custom:') or gripper.startswith('allegro-hand:')}">
+    <xacro:unless value="${gripper in [None, 'onrobot-rg2', 'onrobot-rg6', 'onrobot-rg6-v2', 'weiss-wsg50'] or gripper.startswith('custom:') or gripper.startswith('allegro-hand:')}">
       <xacro:unknown_gripper_type/>
     </xacro:unless>
@@ -25,4 +27,10 @@
         <origin xyz="${pose['x']} ${pose['y']} ${pose['z']}" rpy="${pose['roll']} ${pose['pitch']} ${pose['yaw']}"/>
       </xacro:onrobot_rg>
+    </xacro:if>
+    <!-- if weiss-wsg50 -->
+    <xacro:if value="${gripper == 'weiss-wsg50'}">
+      <xacro:wsg_50_xacro name="${prefix}wsg50" parent="${parent}" finger_length="0.023" finger_tip="0.0" >
+        <origin xyz="${pose['x']} ${pose['y']} ${pose['z']}" rpy="${pose['roll']} ${pose['pitch']} ${pose['yaw']}"/>
+      </xacro:wsg_50_xacro>
     </xacro:if>
     <!-- if allegro-hand -->

Commit message: pr review

File: prl_ur5_description/urdf/_gripper.urdf.xacro (robot description, xacro)
@@ -3,7 +3,9 @@
   <!-- onrobot RG2(6) -->
   <xacro:include filename="$(find onrobot_description)/urdf/onrobot_rg.urdf.xacro"/>
+  <!-- weiss wsg50-->
+  <xacro:include filename="$(find wsg50_simulation)/urdf/wsg_50.urdf.xacro"/>
   <xacro:macro name="gripper" params="gripper prefix parent pose hardware_interface gz_sim">
     <!-- check gripper type -->
-    <xacro:unless value="${gripper in [None, 'onrobot-rg2', 'onrobot-rg6', 'onrobot-rg6-v2'] or gripper.startswith('custom:') or gripper.startswith('allegro-hand:')}">
+    <xacro:unless value="${gripper in [None, 'onrobot-rg2', 'onrobot-rg6', 'onrobot-rg6-v2', 'weiss-wsg50'] or gripper.startswith('custom:') or gripper.startswith('allegro-hand:')}">
       <xacro:unknown_gripper_type/>
     </xacro:unless>
@@ -25,4 +27,10 @@
         <origin xyz="${pose['x']} ${pose['y']} ${pose['z']}" rpy="${pose['roll']} ${pose['pitch']} ${pose['yaw']}"/>
       </xacro:onrobot_rg>
+    </xacro:if>
+    <!-- if weiss-wsg50 -->
+    <xacro:if value="${gripper == 'weiss-wsg50'}">
+      <xacro:wsg_50_xacro name="${prefix}wsg50" parent="${parent}" finger_length="0.023" finger_tip="0.0">
+        <origin xyz="${pose['x']} ${pose['y']} ${pose['z']}" rpy="${pose['roll']} ${pose['pitch']} ${pose['yaw']}"/>
+      </xacro:wsg_50_xacro>
     </xacro:if>
     <!-- if allegro-hand -->

File: prl_ur5_description/urdf/workbench_ur5.urdf.xacro (robot description, xacro)
@@ -76,5 +76,5 @@
                  pose="${left['arm_pose']}"
                  sensor="false"
-                 gripper="${left.get('gripper')}"
+                 gripper="weiss-wsg50"
                  gripper_pose="${left.get('gripper_pose')}"
                  hardware_interface="hardware_interface/PositionJointInterface"
@@ -88,5 +88,5 @@
                  pose="${right['arm_pose']}"
                  sensor="false"
-                 gripper="onrobot-rg6"
+                 gripper="weiss-wsg50"
                  gripper_pose="${right.get('gripper_pose')}"
                  hardware_interface="hardware_interface/PositionJointInterface"

File: prl_ur5_gazebo/urdf/_ft300_gazebo.urdf.xacro (robot description, xacro)
@@ -21,5 +21,5 @@
         </xacro:robotiq_ft300>
         <!-- robotiq sensor hardware ros2 control-->
-        <xacro:robotiq_fts_ros2_control
+        <!-- <xacro:robotiq_fts_ros2_control
             name="${prefix}ft300"
             use_fake_mode="${use_fake_mode}"
@@ -28,5 +28,5 @@
             ftdi_id="${ftdi_id}"
             tf_prefix="${prefix}"
-        />
+        /> -->
         <!-- enable force_torque sensor -->
         <gazebo reference="${prefix}measurment_joint">
@@ -43,6 +43,25 @@
             </sensor>
         </gazebo>
+        <gazebo>
+            <plugin filename="ignition-gazebo-forcetorque-system" name="ignition::gazebo::systems::ForceTorque">
+                <updateRate>100.0</updateRate>
+                <topicName>${prefix}ft_wrench</topicName>
+                <jointName>${prefix}measurment_joint</jointName>
+                <noise>
+                <type>gaussian</type>
+                <mean>0.0</mean>
+                <stddev>0.003</stddev>
+                </noise>
+            </plugin>
+        </gazebo>
+        <!-- override link properties -->
+        <gazebo reference="${prefix}ft300_sensor">
+            <material>Gazebo/Black</material>
+            <selfCollide>true</selfCollide>
+        </gazebo>
+        <gazebo reference="${prefix}ft300_mounting_plate">
+            <material>Gazebo/Grey</material>
+            <selfCollide>true</selfCollide>
+        </gazebo>
     </xacro:macro>
 </robot>
-<!-- [gazebo-3] [ERROR] [1740999000.657453490] [controller_manager]: Caught exception of type : St13runtime_error while claiming the state interfaces.
- Can't activate controller 'robotiq_force_torque_sensor_broadcaster': State interface with key 'left_robotiq_ft_sensor/force.x' does not exist -->

File: prl_ur5_gazebo/urdf/ur5_complete_arm_gazebo.urdf.xacro (robot description, xacro)
@@ -4,4 +4,8 @@
     <xacro:include filename="$(find ur_description)/urdf/ur_macro.xacro"/>
     <xacro:include filename="$(find ur_simulation_gz)/urdf/ur_gz.ros2_control.xacro" />
+    <!-- force sensor-->
+    <xacro:include filename="$(find prl_ur5_gazebo)/urdf/_ft300_gazebo.urdf.xacro"/>
+    <!-- gripper -->
+    <xacro:include filename="$(find prl_ur5_description)/urdf/_gripper.urdf.xacro"/>
     <xacro:macro name="ur5" params="
         name:=ur
@@ -44,4 +48,9 @@
             transmission_hw_interface="${hw_interface}"
         />
+        <!-- force sensor -->
+        <xacro:ft300_gazebo
+            prefix="${prefix}"
+            parent="tool0"
+        />
     </xacro:macro>
 </robot>

File: prl_ur5_gazebo/urdf/workbench_gazebo.urdf.xacro (robot description, xacro)
@@ -98,8 +98,5 @@
   <gazebo>
       <plugin filename="gz_ros2_control-system" name="gz_ros2_control::GazeboSimROS2ControlPlugin">
-      <parameters>$(find prl_ur5_gazebo)/config/dual_ur_controller.yaml</parameters>
-      </plugin>
-      <plugin filename="ignition-gazebo-forcetorque-system" name="ignition::gazebo::systems::ForceTorque">
-      <parameters>$(find prl_ur5_gazebo)/config/ft300_controller.yaml</parameters>
+      <parameters>$(find prl_ur5_control)/config/dual_ur_controller.yaml</parameters>
       </plugin>
   </gazebo>

Commit message: wsg integrate in workbench simulation

File: prl_ur5_description/urdf/_gripper.urdf.xacro (robot description, xacro)
@@ -4,5 +4,5 @@
   <xacro:include filename="$(find onrobot_description)/urdf/onrobot_rg.urdf.xacro"/>
   <!-- weiss wsg50-->
-  <xacro:include filename="$(find wsg_50_simulation)/urdf/wsg_50.urdf.xacro"/>
+  <xacro:include filename="$(find wsg50_simulation)/urdf/wsg_50.urdf.xacro"/>
   <xacro:macro name="gripper" params="gripper prefix parent pose hardware_interface gz_sim">
     <!-- check gripper type -->
@@ -30,5 +30,5 @@
     <!-- if weiss-wsg50 -->
     <xacro:if value="${gripper == 'weiss-wsg50'}">
-      <xacro:wsg_50_xacro name="${prefix}wsg50" parent="${parent}" finger_length="0.023" finger_tip="0.0" >
+      <xacro:wsg_50_xacro name="${prefix}wsg50" parent="${parent}" finger_length="0.023" finger_tip="0.0">
         <origin xyz="${pose['x']} ${pose['y']} ${pose['z']}" rpy="${pose['roll']} ${pose['pitch']} ${pose['yaw']}"/>
       </xacro:wsg_50_xacro>

File: wsg50_simulation/urdf/wsg50.urdf.xacro (robot description, xacro)
@@ -4,5 +4,5 @@
     <xacro:include filename="$(find wsg50_simulation)/urdf/wsg_50.urdf.xacro" />
     <link name="base_link"/>
-    <xacro:wsg_50_xacro name="wsg50" parent="base_link" finger_length="0.023" finger_tip="0.0" >
+    <xacro:wsg_50_xacro name="wsg50" parent="base_link" finger_length="0.023" finger_tip="0.0">
         <origin xyz="0 0 0.1" rpy="0 0 0"/>
     </xacro:wsg_50_xacro>

File: wsg50_simulation/urdf/wsg_50.urdf.xacro (robot description, xacro)
@@ -52,5 +52,5 @@
   <!-- GRIPPER LEFT -->
   <joint name="${name}_base_joint_gripper_left" type="prismatic">
-     <limit lower="-0.055" upper="-0.0027" effort="1.0" velocity="1.0"/>
+     <limit lower="-0.055" upper="-0.003" effort="1.0" velocity="1.0"/>
      <origin xyz="0 0 0" rpy="0 0 0" />      <!--origin xyz="-0.0067 0 0.049" rpy="0 0 0" /-->
      <parent link="${name}_base_link"/>
@@ -102,5 +102,5 @@
      <parent link="${name}_gripper_left"/>
      <child link="${name}_finger_left" />
-     <dynamics friction="100" damping="100" />
+     <!-- <dynamics friction="100" damping="100" /> -->
      <axis xyz="1 0 0"/>
      <limit effort="100" velocity="100"/>
@@ -137,5 +137,5 @@
   <!-- GRIPPER RIGHT -->
   <joint name="${name}_base_joint_gripper_right" type="prismatic">
-     <limit lower="0.0027" upper="0.055" effort="1.0" velocity="1.0"/>
+     <limit lower="0.003" upper="0.055" effort="1.0" velocity="1.0"/>
      <origin xyz="0 0 0" rpy="0 0 3.14159" />
      <parent link="${name}_base_link"/>
@@ -187,5 +187,5 @@
      <parent link="${name}_gripper_right"/>
      <child link="${name}_finger_right" />
-     <dynamics friction="100" damping="100" />
+     <!-- <dynamics friction="100" damping="100" /> -->
      <axis xyz="1 0 0"/>
      <limit effort="100" velocity="100"/>
@@ -228,5 +228,8 @@
         <command_interface name="velocity"/>
         <state_interface name="velocity"/>
-        <state_interface name="position"/>
+        <state_interface name="position">
+        <!-- initial position for the mock system and simulation to avoid fingers spanning into other parts-->
+            <param name="initial_value">0.025</param>
+        </state_interface>
     </joint>
     <joint name="${name}_base_joint_gripper_left">
@@ -234,12 +237,15 @@
         <command_interface name="position"/>
         <state_interface name="position"/>
-        <state_interface name="velocity"/>
+        <state_interface name="position">
+        <!-- initial position for the mock system and simulation to avoid fingers spanning into other parts -->
+            <param name="initial_value">-0.025</param>
+        </state_interface>
     </joint>
   </ros2_control>
-  <gazebo>
+  <!-- <gazebo>
       <plugin filename="gz_ros2_control-system" name="gz_ros2_control::GazeboSimROS2ControlPlugin">
       <parameters>$(find wsg50_simulation)/controllers/wsg50_driver.yaml</parameters>
       </plugin>
-  </gazebo>
+  </gazebo> -->
 </xacro:macro>
 </robot>

Commit message: Interchangeable gripper in Moveit + WSG "clean" integration

File: prl_ur5_description/urdf/_gripper.urdf.xacro (robot description, xacro)
@@ -29,5 +29,5 @@
     <xacro:if value="${gripper == 'weiss-wsg50'}">
       <xacro:include filename="$(find wsg_50_simulation)/urdf/wsg_50.urdf.xacro"/>
-      <xacro:wsg_50_xacro prefix="${prefix}gripper" parent="${parent}" finger_length="0.023" finger_tip="0.0">
+      <xacro:wsg_50_xacro prefix="${prefix}gripper" parent="${parent}" finger_length="0.023" finger_tip="0.0" real_hardware="${not gz_sim}" sim_standalone="false">
         <origin xyz="${pose['x']} ${pose['y']} ${pose['z']}" rpy="${pose['roll']} ${pose['pitch']} ${pose['yaw']}"/>
       </xacro:wsg_50_xacro>

File: prl_ur5_moveit/config/mantis.ros2_control.xacro (robot description, xacro)
@@ -1,5 +1,5 @@
 <?xml version="1.0"?>
 <robot xmlns:xacro="http://www.ros.org/wiki/xacro">
-    <xacro:macro name="ur5_ros2_control" params="name initial_positions_file">
+    <xacro:macro name="mantis_ros2_control" params="name initial_positions_file">
         <xacro:property name="initial_positions" value="${xacro.load_yaml(initial_positions_file)['initial_positions']}"/>
         <ros2_control name="${name}" type="system">

File: prl_ur5_moveit/config/mantis.urdf.xacro (robot description, xacro)
@@ -1,9 +1,9 @@
 <?xml version="1.0"?>
-<robot xmlns:xacro="http://www.ros.org/wiki/xacro" name="ur5">
+<robot xmlns:xacro="http://www.ros.org/wiki/xacro" name="mantis">
     <xacro:arg name="initial_positions_file" default="initial_positions.yaml" />
     <!-- Import ur5 urdf file -->
     <xacro:include filename="$(find prl_ur5_description)/urdf/mantis.urdf.xacro" />
     <!-- Import control_xacro -->
-    <xacro:include filename="ur5.ros2_control.xacro" />
-    <xacro:ur5_ros2_control name="FakeSystem" initial_positions_file="$(arg initial_positions_file)"/>
+    <xacro:include filename="mantis.ros2_control.xacro" />
+    <xacro:mantis_ros2_control name="FakeSystem" initial_positions_file="$(arg initial_positions_file)"/>
 </robot>
