Commit message: urdf integration

File: prl_ur5_description/urdf/_fixed_cameras.urdf.xacro (robot description, xacro)
@@ -4,4 +4,5 @@
     <!-- It is assumed that this file has already been included somewhere else (e.g. in _ur5.urdf.xacro) -->
     <xacro:include filename="$(find prl_ur5_description)/urdf/_camera_sensor.urdf.xacro"/>
+    <xacro:include filename="$(find orbbec_description)/urdf/femto_bolt.urdf.xacro"/>
     <!-- Build fixed camera with their support from one file -->
     <xacro:macro name="fixed_cameras" params="parent fixed_cameras_file turn_on:=false">
@@ -23,5 +24,5 @@
         <!-- Spawn camera -->
             <!-- check camera type -->
-        <xacro:unless value="${camera['type'] in ['realsense-d435i']}">
+        <xacro:unless value="${camera['type'] in ['realsense-d435i', 'femto-mega']}">
             <xacro:unknown_camera_type/>
         </xacro:unless>
@@ -42,4 +43,9 @@
                                  pose="${dict(x=0.0325, y=0.0125, z=-0.0106, roll=pi/2.0, pitch=-pi/2.0, yaw=0)}"
                                 />
+        </xacro:if>
+        <xacro:if value="${camera['type'] == 'femto-mega'}">
+            <xacro:femto_bolt prefix="${camera['name_prefix']}_camera" parent="${parent}" use_nominal_extrinsics="true">
+                <origin xyz="${camera['pose']['x']} ${camera['pose']['y']} ${camera['pose']['z']}" rpy="${camera['pose']['roll']} ${camera['pose']['pitch']} ${camera['pose']['yaw']}"/>
+            </xacro:femto_bolt>
         </xacro:if>
         <!-- Numerical dimensions for the fixtures -->
