Commit message: pr review coorection (remove all gazebo parts)

File: prl_ur5_description/urdf/_camera_sensor.urdf.xacro (robot description, xacro)
@@ -3,5 +3,4 @@
   <!-- realsense d435i -->
   <xacro:include filename="$(find realsense2_description)/urdf/_d435i.urdf.xacro"/>
-  <xacro:include filename="$(find prl_ur5_description)/urdf/_d435.gazebo.xacro"/>
   <xacro:macro name="camera_sensor" params="prefix parent camera pose turn_on:=false">
     <!-- check camera type -->
@@ -14,5 +13,4 @@
         <origin xyz="${pose['x']} ${pose['y']} ${pose['z']}" rpy="${pose['roll']} ${pose['pitch']} ${pose['yaw']}"/>
       </xacro:sensor_d435i>
-      <xacro:gazebo_d435 name="${prefix}camera" turn_on="${turn_on}" visualize="true"/>
     </xacro:if>
   </xacro:macro>

File: prl_ur5_description/urdf/_fixed_cameras.urdf.xacro (robot description, xacro)
@@ -89,14 +89,4 @@
             </collision>
         </link>
-        <gazebo reference="fixed_camera_${number}_bb">
-            <visual>
-            <material>
-                <ambient>0.1 0.5 0.5 0.2</ambient>
-                <diffuse>0.1 0.5 0.1 0.2</diffuse>
-                <specular>0.1 0.1 0.1 0.2</specular>
-                <emissive>0.0 0.0 0.0 0.0</emissive>
-            </material>
-            </visual>
-        </gazebo>
         <joint name="fixed_camera_${number}_bb_joint" type="fixed">
             <parent link = "${parent}"/>
@@ -118,7 +108,4 @@
             </collision>
         </link>
-        <gazebo reference="fixed_camera_${number}_sj">
-                <material>Gazebo/BlueGlow</material>
-        </gazebo>
         <joint name="fixed_camera_${number}_sj_joint" type="fixed">
             <parent link = "fixed_camera_${number}_bb"/>
@@ -140,7 +127,4 @@
             </collision>
         </link>
-        <gazebo reference="fixed_camera_${number}_vt">
-                <material>Gazebo/BlueGlow</material>
-        </gazebo>
         <joint name="fixed_camera_${number}_vt_joint" type="fixed">
             <parent link = "fixed_camera_${number}_sj"/>
@@ -162,7 +146,4 @@
             </collision>
         </link>
-        <gazebo reference="fixed_hr_${number}">
-                <material>Gazebo/BlueGlow</material>
-        </gazebo>
         <joint name="fixed_hr_${number}_fix" type="fixed">
             <parent link = "fixed_camera_${number}_vt"/>

Commit message: maj package

File: prl_ur5_description/urdf/_camera_sensor.urdf.xacro (robot description, xacro)
@@ -3,4 +3,5 @@
   <!-- realsense d435i -->
   <xacro:include filename="$(find realsense2_description)/urdf/_d435i.urdf.xacro"/>
+  <xacro:include filename="$(find prl_ur5_description)/urdf/_d435_gazebo.urdf.xacro"/>
   <xacro:macro name="camera_sensor" params="prefix parent camera pose turn_on:=false">
     <!-- check camera type -->
@@ -13,4 +14,5 @@
         <origin xyz="${pose['x']} ${pose['y']} ${pose['z']}" rpy="${pose['roll']} ${pose['pitch']} ${pose['yaw']}"/>
       </xacro:sensor_d435i>
+      <xacro:gazebo_d435 name="${prefix}camera" turn_on="${turn_on}"/>
     </xacro:if>
   </xacro:macro>

File: prl_ur5_description/urdf/ur5_complete_arm.urdf.xacro (robot description, xacro)
@@ -61,4 +61,32 @@
             gz_sim="${gz_sim}"
         />
+        <!-- tool frame -->
+        <link name="${prefix}tool"/>
+        <joint name="${prefix}tool_joint" type="fixed">
+            <origin xyz="0 0 0" rpy="0 0 ${-pi}"/>
+            <parent link="${prefix}robotiq_ft_frame_id"/>
+            <child link="${prefix}tool"/>
+        </joint>
+        <!-- gripper -->
+        <xacro:gripper gripper="${gripper}" prefix='${prefix}' parent="${prefix}tool" pose="${gripper_pose}" hardware_interface="${hw_interface}" gz_sim="${gz_sim}"/>
+        <!-- Right angle connector -->
+        <link name="${prefix}wrist_connector_link">
+        <visual>
+            <geometry>
+                <mesh filename="file://$(find prl_ur5_description)/model/RG_connector_simple.stl"/>
+            </geometry>
+            <material name="connector_green"><color rgba="0.2 0.8 0 1"/></material>
+        </visual>
+        <collision>
+            <geometry>
+                <mesh filename="file://$(find prl_ur5_description)/model/RG_connector_simple_convex.stl"/>
+            </geometry>
+        </collision>
+        </link>
+        <joint name="${prefix}wrist_connector" type="fixed">
+        <origin xyz="0 -0.0375 -0.02" rpy="1.5708 0 0"/>
+        <parent link="${prefix}wrist_3_link"/>
+        <child link="${prefix}wrist_connector_link"/>
+        </joint>
     </xacro:macro>
 </robot>

File: wsg50_simulation/urdf/wsg_50.urdf.xacro (robot description, xacro)
@@ -5,242 +5,273 @@
                     Use e.g. for single contact point tip on finger. (default 0) -->
 <xacro:macro name="wsg_50_xacro" params="name parent finger_length finger_tip *origin">
- <joint name="${name}_anterior_gripper_joint" type="fixed">
-    <xacro:insert_block name="origin"/>
-    <parent link="${parent}"/>
-    <child link="${name}_base_link"/>
- </joint>
-<!-- BASE LINK -->
- <link name="${name}_base_link">
-      <inertial>
-          <mass value="0.25" />
-          <origin xyz="0 0 0" />
-     	  <!--inertia ixx="1.0" ixy="0.0" ixz="0.0"
-               iyy="100.0" iyz="0.0"
-               izz="1.0" /-->
-      	  <inertia  ixx="1.0" ixy="0.0"  ixz="0.0"  iyy="1.0"  iyz="0.0"  izz="1.0" />
-      </inertial>
-      <visual>
-          <origin xyz="0.0 0 0" rpy="0 0 0" />
-          <geometry>
-             <mesh filename="file://$(find wsg50_simulation)/meshes/WSG50_110.stl" scale="1 1 1"/>
-	     <!--box size="0.146 0.05 0.0735"/-->
-          </geometry>
-          <!-- <material name="grey">-->
-            <material name="Robotiq-LightGrey">
-            <color rgba="1 1 1 1"/>
-          </material>
-      </visual>
-      <collision>
-          <origin xyz="0.0 0 0" rpy="0 0 0" />
-          <geometry>
-	     <!--box size="0.146 0.05 0.0735"/-->
-             <mesh filename="file://$(find wsg50_simulation)/meshes/WSG50_110.stl" scale="1 1 1"/>
-         </geometry>
-     </collision>
-  </link>
-  <gazebo reference="${name}_base_link">
-    <material>Gazebo/Grey</material>
-    <turnGravityOff>false</turnGravityOff>
-  </gazebo>
-  <joint name="${name}_center_joint" type="fixed">
-     <origin xyz="0 0 ${finger_length}" rpy="0 0 0" />      <!--origin xyz="-0.0067 0 0.049" rpy="0 0 0" /-->
-     <parent link="${name}_base_link"/>
-     <child link="${name}_center" />
-  </joint>
-  <link name="${name}_center">
-  </link>
-  <!-- GRIPPER LEFT -->
-  <joint name="${name}_base_joint_gripper_left" type="prismatic">
-     <limit lower="-0.055" upper="-0.003" effort="1.0" velocity="1.0"/>
-     <origin xyz="0 0 0" rpy="0 0 0" />      <!--origin xyz="-0.0067 0 0.049" rpy="0 0 0" /-->
-     <parent link="${name}_base_link"/>
-     <child link="${name}_gripper_left" />
-     <!-- <dynamics friction="100" damping="100" /> -->
-     <axis xyz="1 0 0"/>
-     <limit effort="100" velocity="100"/>
-  </joint>
-  <transmission name="${name}_base_trans_left" type="pr2_mechanism_model/SimpleTransmission">
-     <actuator name="${name}_base_motor_left" />
-     <joint name="${name}_base_joint_gripper_left" />
-     <mechanicalReduction>1</mechanicalReduction>
-     <motorTorqueConstant>1</motorTorqueConstant>
-  </transmission>
-  <link name="${name}_gripper_left">
-      <inertial>
-          <mass value="0.1" />
-          <origin xyz="0 0 0" />
-      <inertia ixx="1.0" ixy="0.0" ixz="0.0"
-               iyy="1.0" iyz="0.0"
-               izz="1.0" />
-      </inertial>
-      <visual>
-          <origin xyz="0.0 0 0" rpy="0 0 0" />
-          <geometry>
-             <mesh filename="file://$(find wsg50_simulation)/meshes/GUIDE_WSG50_110.stl" scale="0.001 0.001 0.001"/>
-	     <!--box size="0.0175 0.03 0.024"/-->
-          </geometry>
-          <material name="black">
-		<color rgba="0 0 0 1"/>
-      	  </material>
-      </visual>
-      <collision>
-          <origin xyz="0 0 0" rpy="0 0 0" />
-          <geometry>
-	     <!--box size="0.0175 0.03 0.024"/-->
-             <mesh filename="file://$(find wsg50_simulation)/meshes/GUIDE_WSG50_110.stl" scale="0.001 0.001 0.001"/>
-         </geometry>
-     </collision>
-     <contact_coefficients kd="1.0" kp="1000.0" mu="0"/>
-  </link>
-  <gazebo reference="${name}_gripper_left">
-    <material>Gazebo/Blue</material>
-    <turnGravityOff>false</turnGravityOff>
-  </gazebo>
-  <!-- LEFT FINGER -->
-  <joint name="${name}_guide_joint_finger_left" type="fixed">
-     <origin xyz="${finger_tip} 0 ${finger_length}" rpy="0 0 0" />
-     <parent link="${name}_gripper_left"/>
-     <child link="${name}_finger_left" />
-     <!-- <dynamics friction="100" damping="100" /> -->
-     <axis xyz="1 0 0"/>
-     <limit effort="100" velocity="100"/>
-  </joint>
-  <link name="${name}_finger_left">
-      <inertial>
-          <mass value="0.1" />
-          <origin xyz="0 0 0" />
-      <inertia ixx="1.0" ixy="0.0" ixz="0.0"
-               iyy="1.0" iyz="0.0"
-               izz="1.0" />
-      </inertial>
-      <visual>
-          <origin xyz="0.0 0 0" rpy="0 0 0" />
-          <geometry>
-             <mesh filename="file://$(find wsg50_simulation)/meshes/WSG-FMF.stl" scale="0.001 0.001 0.001"/>
-          </geometry>
-          <material name="black">
-		<color rgba="0 0 0 1"/>
-      	  </material>
-      </visual>
-      <collision>
-          <origin xyz="0 0 0" rpy="0 0 0" />
-          <geometry>
-             <mesh filename="file://$(find wsg50_simulation)/meshes/WSG-FMF.stl" scale="0.001 0.001 0.001"/>
-         </geometry>
-     </collision>
-     <contact_coefficients kd="1.0" kp="1000.0" mu="0"/>
-  </link>
-  <gazebo reference="${name}_finger_left">
-    <material>Gazebo/Blue</material>
-    <turnGravityOff>false</turnGravityOff>
-  </gazebo>
-  <!-- GRIPPER RIGHT -->
-  <joint name="${name}_base_joint_gripper_right" type="prismatic">
-     <limit lower="0.003" upper="0.055" effort="1.0" velocity="1.0"/>
-     <origin xyz="0 0 0" rpy="0 0 3.14159" />
-     <parent link="${name}_base_link"/>
-     <child link="${name}_gripper_right" />
-     <axis xyz="-1 0 0"/>
-     <!-- <dynamics friction="100" damping="100" /> -->
-     <limit effort="100" velocity="100"/>
-  </joint>
-  <transmission name="${name}_base_trans_right" type="pr2_mechanism_model/SimpleTransmission">
-     <actuator name="${name}_base_motor_right" />
-     <joint name="${name}_base_joint_gripper_right" />
-     <mechanicalReduction>1</mechanicalReduction>
-     <motorTorqueConstant>1</motorTorqueConstant>
-  </transmission>
-    <link name="${name}_gripper_right">
-      <inertial>
-          <mass value="0.1" />
-          <origin xyz="0 0 0" />
-      <inertia ixx="1.0" ixy="0.0" ixz="0.0"
-               iyy="1.0" iyz="0.0"
-               izz="1.0" />
-      </inertial>
-      <visual>
-          <origin xyz="0.0 0 0" rpy="0 0 0" />
-          <geometry>
-             <mesh filename="file://$(find wsg50_simulation)/meshes/GUIDE_WSG50_110.stl" scale="0.001 0.001 0.001"/>
-	     <!--box size="0.0175 0.03 0.024"/-->
-          </geometry>
-          <material name="black">
-		    <color rgba="0 0 0 1"/>
-      	  </material>
-      </visual>
-      <collision>
-          <origin xyz="0 0 0" rpy="0 0 0" />
-          <geometry>
-	     <!--box size="0.0175 0.03 0.024"/-->
-             <mesh filename="file://$(find wsg50_simulation)/meshes/GUIDE_WSG50_110.stl" scale="0.001 0.001 0.001"/>
-         </geometry>
-     </collision>
-     <contact_coefficients kd="1.0" kp="1000.0" mu="0"/>
-  </link>
-  <gazebo reference="gripper_right">
-    <material>Gazebo/White</material>
-    <turnGravityOff>false</turnGravityOff>
-  </gazebo>
-  <!-- RIGHT FINGER -->
-  <joint name="${name}_guide_joint_finger_right" type="fixed">
-     <origin xyz="${finger_tip} 0 ${finger_length}" rpy="0 0 0" />
-     <parent link="${name}_gripper_right"/>
-     <child link="${name}_finger_right" />
-     <!-- <dynamics friction="100" damping="100" /> -->
-     <axis xyz="1 0 0"/>
-     <limit effort="100" velocity="100"/>
-  </joint>
-  <link name="${name}_finger_right">
-      <inertial>
-          <mass value="0.1" />
-          <origin xyz="0 0 0" />
-      <inertia ixx="1.0" ixy="0.0" ixz="0.0"
-               iyy="1.0" iyz="0.0"
-               izz="1.0" />
-      </inertial>
-      <visual>
-          <origin xyz="0.0 0 0" rpy="0 0 0" />
-          <geometry>
-             <mesh filename="file://$(find wsg50_simulation)/meshes/WSG-FMF.stl" scale="0.001 0.001 0.001"/>
-          </geometry>
-          <material name="black">
-		<color rgba="0 0 0 1"/>
-      	  </material>
-      </visual>
-      <collision>
-          <origin xyz="0 0 0" rpy="0 0 0" />
-          <geometry>
-             <mesh filename="file://$(find wsg50_simulation)/meshes/WSG-FMF.stl" scale="0.001 0.001 0.001"/>
-         </geometry>
-     </collision>
-     <contact_coefficients kd="1.0" kp="1000.0" mu="0"/>
-  </link>
-  <gazebo reference="${name}_finger_right">
-    <material>Gazebo/White</material>
-    <turnGravityOff>false</turnGravityOff>
-  </gazebo>
-  <ros2_control name="${name}" type="actuator">
-    <hardware>
-        <plugin>gz_ros2_control/GazeboSimSystem</plugin>
-    </hardware>
-    <joint name="${name}_base_joint_gripper_right">
-        <command_interface name="position"/>
-        <command_interface name="velocity"/>
-        <state_interface name="velocity"/>
-        <state_interface name="position">
-        <!-- initial position for the mock system and simulation to avoid fingers spanning into other parts-->
-            <param name="initial_value">0.025</param>
-        </state_interface>
-    </joint>
-    <joint name="${name}_base_joint_gripper_left">
-        <command_interface name="velocity"/>
-        <command_interface name="position"/>
-        <state_interface name="position"/>
-        <state_interface name="position">
-        <!-- initial position for the mock system and simulation to avoid fingers spanning into other parts -->
-            <param name="initial_value">-0.025</param>
-        </state_interface>
-    </joint>
-  </ros2_control>
+    <joint name="${name}_mounting_plate_joint" type="fixed">
+        <xacro:insert_block name="origin"/>
+        <parent link="${parent}"/>
+        <child link="${name}_mounting_plate"/>
+    </joint>
+    <link name="${name}_mounting_plate">
+        <inertial>
+            <mass value="0.25" />
+            <origin xyz="0 0 -0.1" />
+        	  <inertia  ixx="1.0" ixy="0.0"  ixz="0.0"  iyy="1.0"  iyz="0.0"  izz="1.0" />
+        </inertial>
+        <visual>
+            <origin xyz="0.0 0 0" rpy="0 0 0" />
+            <geometry>
+                 <mesh filename="file://$(find wsg50_simulation)/meshes/FL_ISO50_WSG50.stl" scale="0.001 0.001 0.001"/>
+            </geometry>
+            <material name="black">
+                <color rgba="0 0 0 1"/>
+            </material>
+        </visual>
+        <collision>
+            <origin xyz="0.0 0 0" rpy="0 0 0" />
+            <geometry>
+                 <mesh filename="file://$(find wsg50_simulation)/meshes/FL_ISO50_WSG50.stl" scale="0.001 0.001 0.001"/>
+            </geometry>
+         </collision>
+    </link>
+    <!-- <gazebo reference="${name}_mounting_plate">
+        <material>Gazebo/Grey</material>
+        <turnGravityOff>true</turnGravityOff>
+    </gazebo> -->
+    <joint name="${name}_anterior_gripper_joint" type="fixed">
+        <parent link="${name}_mounting_plate"/>
+        <child link="${name}_base_link"/>
+        <origin xyz="0 0 0" rpy="0 0 ${pi}" />
+    </joint>
+    <!-- BASE LINK -->
+    <link name="${name}_base_link">
+        <inertial>
+            <mass value="0.25" />
+            <origin xyz="0 0 0" />
+            <!--inertia ixx="1.0" ixy="0.0" ixz="0.0"
+                iyy="100.0" iyz="0.0"
+                izz="1.0" /-->
+            <inertia  ixx="1.0" ixy="0.0"  ixz="0.0"  iyy="1.0"  iyz="0.0"  izz="1.0" />
+        </inertial>
+        <visual>
+            <origin xyz="0.0 0 0" rpy="0 0 0" />
+            <geometry>
+                <mesh filename="file://$(find wsg50_simulation)/meshes/WSG50_110.stl" scale="1 1 1"/>
+            <!--box size="0.146 0.05 0.0735"/-->
+            </geometry>
+            <!-- <material name="grey">-->
+                <material name="Robotiq-LightGrey">
+                <color rgba="1 1 1 1"/>
+            </material>
+        </visual>
+        <collision>
+            <origin xyz="0.0 0 0" rpy="0 0 0" />
+            <geometry>
+            <!--box size="0.146 0.05 0.0735"/-->
+                <mesh filename="file://$(find wsg50_simulation)/meshes/WSG50_110.stl" scale="1 1 1"/>
+            </geometry>
+        </collision>
+    </link>
+    <gazebo reference="${name}_base_link">
+        <material>Gazebo/Grey</material>
+        <turnGravityOff>true</turnGravityOff>
+    </gazebo>
+    <joint name="${name}_center_joint" type="fixed">
+        <origin xyz="0 0 ${finger_length}" rpy="0 0 0" />      <!--origin xyz="-0.0067 0 0.049" rpy="0 0 0" /-->
+        <parent link="${name}_base_link"/>
+        <child link="${name}_center" />
+    </joint>
+    <link name="${name}_center">
+    </link>
+    <!-- GRIPPER LEFT -->
+    <joint name="${name}_base_joint_gripper_left" type="prismatic">
+        <limit lower="-0.055" upper="-0.003" effort="1.0" velocity="1.0"/>
+        <origin xyz="0 0 0" rpy="0 0 0" />      <!--origin xyz="-0.0067 0 0.049" rpy="0 0 0" /-->
+        <parent link="${name}_base_link"/>
+        <child link="${name}_gripper_left" />
+        <!-- <dynamics friction="100" damping="100" /> -->
+        <axis xyz="1 0 0"/>
+        <limit effort="100" velocity="100"/>
+    </joint>
+    <transmission name="${name}_base_trans_left" type="pr2_mechanism_model/SimpleTransmission">
+        <actuator name="${name}_base_motor_left" />
+        <joint name="${name}_base_joint_gripper_left" />
+        <mechanicalReduction>1</mechanicalReduction>
+        <motorTorqueConstant>1</motorTorqueConstant>
+    </transmission>
+    <link name="${name}_gripper_left">
+        <inertial>
+            <mass value="0.1" />
+            <origin xyz="0 0 0" />
+        <inertia ixx="1.0" ixy="0.0" ixz="0.0"
+                iyy="1.0" iyz="0.0"
+                izz="1.0" />
+        </inertial>
+        <visual>
+            <origin xyz="0.0 0 0" rpy="0 0 0" />
+            <geometry>
+                <mesh filename="file://$(find wsg50_simulation)/meshes/GUIDE_WSG50_110.stl" scale="0.001 0.001 0.001"/>
+            <!--box size="0.0175 0.03 0.024"/-->
+            </geometry>
+            <material name="black">
+            <color rgba="0 0 0 1"/>
+            </material>
+        </visual>
+        <collision>
+            <origin xyz="0 0 0" rpy="0 0 0" />
+            <geometry>
+            <!--box size="0.0175 0.03 0.024"/-->
+                <mesh filename="file://$(find wsg50_simulation)/meshes/GUIDE_WSG50_110.stl" scale="0.001 0.001 0.001"/>
+            </geometry>
+        </collision>
+        <contact_coefficients kd="1.0" kp="1000.0" mu="0"/>
+    </link>
+    <gazebo reference="${name}_gripper_left">
+        <material>Gazebo/Blue</material>
+        <turnGravityOff>true</turnGravityOff>
+    </gazebo>
+    <!-- LEFT FINGER -->
+    <joint name="${name}_guide_joint_finger_left" type="fixed">
+        <origin xyz="${finger_tip} 0 ${finger_length}" rpy="0 0 0" />
+        <parent link="${name}_gripper_left"/>
+        <child link="${name}_finger_left" />
+        <!-- <dynamics friction="100" damping="100" /> -->
+        <axis xyz="1 0 0"/>
+        <limit effort="100" velocity="100"/>
+    </joint>
+    <link name="${name}_finger_left">
+        <inertial>
+            <mass value="0.1" />
+            <origin xyz="0 0 0" />
+        <inertia ixx="1.0" ixy="0.0" ixz="0.0"
+                iyy="1.0" iyz="0.0"
+                izz="1.0" />
+        </inertial>
+        <visual>
+            <origin xyz="0.0 0 0" rpy="0 0 0" />
+            <geometry>
+                <mesh filename="file://$(find wsg50_simulation)/meshes/WSG-FMF.stl" scale="0.001 0.001 0.001"/>
+            </geometry>
+            <material name="black">
+            <color rgba="0 0 0 1"/>
+            </material>
+        </visual>
+        <collision>
+            <origin xyz="0 0 0" rpy="0 0 0" />
+            <geometry>
+                <mesh filename="file://$(find wsg50_simulation)/meshes/WSG-FMF.stl" scale="0.001 0.001 0.001"/>
+            </geometry>
+        </collision>
+        <contact_coefficients kd="1.0" kp="1000.0" mu="0"/>
+    </link>
+    <gazebo reference="${name}_finger_left">
+        <material>Gazebo/Blue</material>
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