Commit message: orbbec urdf correction

File: prl_ur5_description/urdf/_camera_sensor.urdf.xacro (robot description, xacro)
@@ -6,5 +6,5 @@
   <xacro:macro name="camera_sensor" params="prefix parent camera pose turn_on:=false">
     <!-- check camera type -->
-    <xacro:unless value="${camera in [None, 'realsense-d435i']}">
+    <xacro:unless value="${camera in ['realsense-d435i', 'femto-mega', None]}">
       <xacro:unknown_camera_type/>
     </xacro:unless>
@@ -16,4 +16,9 @@
       <xacro:gazebo_d435 name="${prefix}camera" turn_on="${turn_on}"/>
     </xacro:if>
+    <xacro:if value="${camera == 'femto-mega'}">
+        <xacro:femto_bolt prefix="${prefix}camera" parent="${parent}" use_nominal_extrinsics="true">
+            <origin xyz="${pose['x']} ${pose['y']} ${pose['z']}" rpy="${pose['roll']} ${pose['pitch']} ${pose['yaw']}"/>
+        </xacro:femto_bolt>
+    </xacro:if>
   </xacro:macro>
 </robot>

File: prl_ur5_description/urdf/_fixed_cameras.urdf.xacro (robot description, xacro)
@@ -23,6 +23,6 @@
     <xacro:macro name="fixed_camera" params="parent number camera turn_on">
         <!-- Spawn camera -->
-            <!-- check camera type -->
-        <xacro:unless value="${camera['type'] in ['realsense-d435i', 'femto-mega']}">
+        <!-- check camera type -->
+        <xacro:unless value="${camera['type'] in ['realsense-d435i', 'femto-mega', 'None']}">
             <xacro:unknown_camera_type/>
         </xacro:unless>
@@ -45,7 +45,15 @@
         </xacro:if>
         <xacro:if value="${camera['type'] == 'femto-mega'}">
-            <xacro:femto_bolt prefix="${camera['name_prefix']}_camera" parent="${parent}" use_nominal_extrinsics="true">
+            <link name="${camera['name_prefix']}_camera_calibration_pose"/>
+            <joint name="${camera['name_prefix']}_camera_calibration_pose_joint" type="fixed">
                 <origin xyz="${camera['pose']['x']} ${camera['pose']['y']} ${camera['pose']['z']}" rpy="${camera['pose']['roll']} ${camera['pose']['pitch']} ${camera['pose']['yaw']}"/>
-            </xacro:femto_bolt>
+                <parent link="${parent}"/>
+                <child link="${camera['name_prefix']}_camera_calibration_pose"/>
+            </joint>
+            <xacro:camera_sensor camera="${camera['type']}"
+                                 prefix="${camera['name_prefix']}_"
+                                 parent="${camera['name_prefix']}_camera_calibration_pose"
+                                 turn_on="${turn_on}"
+                                pose="${dict(x=0.0, y=0.028, z=-0.0106, roll=pi, pitch=.0, yaw=pi/2.0)}" />
         </xacro:if>
         <!-- Numerical dimensions for the fixtures -->
