Commit message: add doc and cameras integration

File: prl_ur5_description/urdf/_d435_gazebo.urdf.xacro (robot description, xacro)
@@ -8,5 +8,5 @@
 <!-- Modified from https://github.com/pal-robotics-forks/realsense -->
 <robot xmlns:xacro="http://ros.org/wiki/xacro">
-  <xacro:macro name="gazebo_d435" params="name turn_on publish_pointcloud:=true visualize:=false" >
+  <xacro:macro name="gazebo_d435" params="name turn_on publish_pointcloud:=true visualize:=true" >
     <!-- Load parameters to model's main link-->
     <xacro:property name="deg_to_rad" value="${pi/180}" />
@@ -108,4 +108,5 @@
             <stddev>0.100</stddev>
           </noise> -->
+          <point_cloud>true</point_cloud>
         </camera>
         <always_on>${turn_on}</always_on>
@@ -115,8 +116,8 @@
     </gazebo>
     <!-- Gazebo creates a link for each sensor, we need to attach them to the main link -->
-    <link name="dual_ur/base_link/${name}_depth"/>
+    <link name="mantis/base_link/${name}_depth"/>
     <joint name="${name}_depth_joint_gz" type="fixed">
       <parent link="${name}_link"/>
-      <child link="dual_ur/base_link/${name}_depth"/>
+      <child link="mantis/base_link/${name}_depth"/>
       <origin xyz="0 0 0" rpy="0 0 0"/>
     </joint>

File: prl_ur5_description/urdf/_gripper.urdf.xacro (robot description, xacro)
@@ -3,4 +3,5 @@
   <!-- onrobot RG2(6) -->
   <xacro:include filename="$(find onrobot_description)/urdf/onrobot_rg.urdf.xacro"/>
+  <!-- Macro to generate gripper -->
   <xacro:macro name="gripper" params="gripper prefix parent pose hardware_interface gz_sim">
     <!-- check gripper type -->

File: prl_ur5_description/urdf/mantis.urdf.xacro (robot description, xacro)
@@ -1,4 +1,4 @@
 <?xml version="1.0"?>
-<robot xmlns:xacro="http://wiki.ros.org/xacro" name="ur5" >
+<robot xmlns:xacro="http://wiki.ros.org/xacro" name="mantis" >
   <!-- Arguments-->
   <xacro:arg name="gz_sim" default="false"/>
@@ -104,4 +104,5 @@
                  network = "${right.get('network')}"
                  />
+  <!-- Gazebosim plugin -->
   <xacro:if value="$(arg gz_sim)">
     <gazebo>

File: prl_ur5_description/urdf/ur5_complete_arm.urdf.xacro (robot description, xacro)
@@ -9,4 +9,5 @@
     <!-- gripper -->
     <xacro:include filename="$(find prl_ur5_description)/urdf/_gripper.urdf.xacro"/>
+    <!-- Macro to define the complete arm -->
     <xacro:macro name="arm" params="
         name:=ur
@@ -33,4 +34,5 @@
         network := ''
         ">
+        <!-- UR5 -->
         <xacro:ur_robot
             name="${prefix}ur"
@@ -48,4 +50,5 @@
         <origin xyz="${pose['x']} ${pose['y']} ${pose['z']}" rpy="${pose['roll']} ${pose['pitch']} ${pose['yaw']}"/>
         </xacro:ur_robot>
+        <!-- ROS2 control if simulation -->
         <xacro:if value="${gz_sim}">
             <ros2_control name="${prefix}ur" type="system">
@@ -59,4 +62,5 @@
             </ros2_control>
         </xacro:if>
+        <!-- ROS2 control if real robot -->
         <xacro:unless value="${gz_sim}">
             <xacro:ur_ros2_control
@@ -77,5 +81,5 @@
             />
         </xacro:unless>
-        <!-- force sensor -->
+        <!-- Force sensor -->
         <xacro:force_sensor
             prefix="${prefix}"
@@ -83,5 +87,5 @@
             gz_sim="${gz_sim}"
         />
-        <!-- tool frame -->
+        <!-- Tool frame -->
         <link name="${prefix}tool"/>
         <joint name="${prefix}tool_joint" type="fixed">
@@ -90,5 +94,5 @@
             <child link="${prefix}tool"/>
         </joint>
-        <!-- gripper -->
+        <!-- Gripper -->
         <xacro:gripper gripper="${gripper}" prefix='${prefix}' parent="${prefix}tool" pose="${gripper_pose}" hardware_interface="${hw_interface}" gz_sim="${gz_sim}"/>
         <!-- Right angle connector -->

Commit message: Update _d435_gazebo.urdf.xacro

File: prl_ur5_description/urdf/_d435_gazebo.urdf.xacro (robot description, xacro)
@@ -27,4 +27,5 @@
       <min_depth>0</min_depth>-->
       <sensor name="${name}_color" type="camera">
+        <gz_frame_id>${name}_color_frame</gz_frame_id>
         <camera name="${name}">
           <horizontal_fov>${69.4*deg_to_rad}</horizontal_fov>
@@ -49,4 +50,5 @@
       </sensor>
       <sensor name="${name}_ired1" type="camera">
+        <gz_frame_id>${name}_infra1_frame</gz_frame_id>
         <camera name="${name}">
           <horizontal_fov>${85.2*deg_to_rad}</horizontal_fov>
@@ -71,4 +73,5 @@
       </sensor>
       <sensor name="${name}_ired2" type="camera">
+        <gz_frame_id>${name}_infra2_frame</gz_frame_id>
         <camera name="${name}">
           <horizontal_fov>${85.2*deg_to_rad}</horizontal_fov>
@@ -93,4 +96,5 @@
       </sensor>
       <sensor name="${name}_depth" type="depth_camera">
+        <gz_frame_id>${name}_depth_frame</gz_frame_id>
         <camera name="${name}">
           <horizontal_fov>${85.2*deg_to_rad}</horizontal_fov>
@@ -115,11 +119,4 @@
       </sensor>
     </gazebo>
-    <!-- Gazebo creates a link for each sensor, we need to attach them to the main link -->
-    <link name="mantis/base_link/${name}_depth"/>
-    <joint name="${name}_depth_joint_gz" type="fixed">
-      <parent link="${name}_link"/>
-      <child link="mantis/base_link/${name}_depth"/>
-      <origin xyz="0 0 0" rpy="0 0 0"/>
-    </joint>
   </xacro:macro>
 </robot>
