Commit message: test markdown blockquote

File: prl_ur5_description/urdf/mantis.urdf.xacro (robot description, xacro)
@@ -6,5 +6,5 @@
   <!-- Setup files -->
   <xacro:arg name="controller_file" default="$(find prl_ur5_control)/config/dual_arm_controller.yaml"/>
-  <xacro:property name="setup_file" value="${xacro.load_yaml('$(find prl_ur5_robot_configuration)/config/standart_setup.yaml')}"/>
+  <xacro:property name="setup_file" value="${xacro.load_yaml('$(find prl_ur5_robot_configuration)/config/standard_setup.yaml')}"/>
   <!-- ur5 arm -->
   <xacro:include filename="$(find prl_ur5_description)/urdf/ur5_complete_arm.urdf.xacro"/>

Commit message: add network config file

File: prl_ur5_description/urdf/mantis.urdf.xacro (robot description, xacro)
@@ -7,4 +7,5 @@
   <xacro:arg name="controller_file" default="$(find prl_ur5_control)/config/dual_arm_controller.yaml"/>
   <xacro:property name="setup_file" value="${xacro.load_yaml('$(find prl_ur5_robot_configuration)/config/standard_setup.yaml')}"/>
+  <xacro:property name="network_file" value="${xacro.load_yaml('$(find prl_ur5_robot_configuration)/config/network_setup.yaml')}"/>
   <!-- ur5 arm -->
   <xacro:include filename="$(find prl_ur5_description)/urdf/ur5_complete_arm.urdf.xacro"/>
@@ -80,4 +81,5 @@
   <!-- Left arm -->
   <xacro:property name="left" value="${setup_file.get('left')}"/>
+  <xacro:property name="left_network" value="${network_file.get('left_network')}"/>
   <xacro:arm prefix="left_"
                  parent="prl_ur5_base"
@@ -91,8 +93,9 @@
                  joint_limits_parameters_file="$(find prl_ur5_robot_configuration)/config/${left.get('arm_joint_limits')}"
                  kinematics_parameters_file="$(find prl_ur5_robot_configuration)/config/${left.get('arm_kinematics')}"
-                 network = "${left.get('network')}"
+                 network = "${left_network}"
                  />
   <!-- Right Arm -->
   <xacro:property name="right" value="${setup_file.get('right')}"/>
+  <xacro:property name="right_network" value="${network_file.get('right_network')}"/>
   <xacro:arm prefix="right_"
                  parent="prl_ur5_base"
@@ -106,5 +109,5 @@
                  joint_limits_parameters_file="$(find prl_ur5_robot_configuration)/config/${right.get('arm_joint_limits')}"
                  kinematics_parameters_file="$(find prl_ur5_robot_configuration)/config/${right.get('arm_kinematics')}"
-                 network = "${right.get('network')}"
+                 network = "${right_network}"
                  />
   <!-- Gazebosim plugin -->
